File: design/can_switcher.brd (EAGLE design)
At the start: 78.4 x 67.3 mm, 49 parts, among them IC1 74HC595D, J3 1X2-3.5MM, U1 NCP1117LPST50T3G, U2 ATMEGA328P-AU, X1 16.000 MHz

Commit message: update design files to get text on proper silkscreen layer; try adding MFG# to various parts
Routing:
- removed copper zone on layer 1, net N$16
